File: schematics/tower-defense/tower-defense.kicad_sch (KiCad schematic)
At the start: 6 parts, among them J1 Conn_01x28_Socket, J2 Conn_01x28_Socket, J3 Barrel_Jack_Switch, J4 Conn_01x16_Socket, J5 Conn_01x04_Socket, U1 COM-09032

Commit message: complete pcb v1
Parts:
- removed U1: COM-09032, Tower_Defense:XDCR_COM-09032, symbol tower_defense:COM-09032
- added C1, C2: 0.1u, Capacitor_SMD:C_0603_1608Metric, symbol Device:C_Small
- added D1: LED_ARGB, Connector_PinSocket_2.54mm:PinSocket_1x04_P2.54mm_Vertical, symbol Device:LED_ARGB
- added D2: LTST-S220KGKT, Tower_Defense:status_led, symbol tower_defense:LTST-S220KGKT
- added J4: Screw_Terminal_01x02, Tower_Defense:screw-terminal, symbol Connector:Screw_Terminal_01x02
- added J5: hub75, Tower_Defense:hub75, symbol tower_defense:hub75
- added J8: Conn_01x03_Socket, Connector_PinSocket_2.54mm:PinSocket_1x03_P2.54mm_Vertical, symbol Connector:Conn_01x03_Socket
- added J9: Conn_01x04_Socket, Connector_PinSocket_2.54mm:PinSocket_1x04_P2.54mm_Vertical, symbol Connector:Conn_01x04_Socket
- added R1, R2, R3: 47, Resistor_SMD:R_0603_1608Metric, symbol Device:R_Small_US
- added R4: 1K, Resistor_SMD:R_0603_1608Metric, symbol Device:R_Small_US
- added SW1: SW_SPDT, Tower_Defense:power_switch, symbol Switch:SW_SPDT
- added U1: joystick, Tower_Defense:joystick, symbol tower_defense:joystick
- added U2, U3: 74AHCT245, Tower_Defense:74HTC245, symbol Adafruit RGB Matrix Bonnet-eagle-import:74LCX245
- renumbered J3 to J1, J4 to J2, J5 to J3, J2 to J6, J1 to J7
Connections:
- net +3.3V: now also U1.H1 (H+), U1.V1 (V+); no longer J6.2 (Pin_2)
- net +5V: now also D2.A, SW1.2 (B); no longer J6.1 (Pin_1), J7.1 (Pin_1)
- net A: now also U3.9 (A8)
- net B: now also J6.22 (Pin_22), U2.9 (A8); no longer J6.17 (Pin_17)
- net B1: now also J6.10 (Pin_10), U3.4 (A3); no longer J6.9 (Pin_9)
- net B2: now also J6.9 (Pin_9), U3.3 (A2); no longer J6.13 (Pin_13)
- net C: now also J6.17 (Pin_17), U2.4 (A3); no longer J6.18 (Pin_18)
- net CLK: now also J6.18 (Pin_18), U2.5 (A4); no longer J6.20 (Pin_20)
- net D: now also J6.21 (Pin_21), U2.8 (A7); no longer J6.19 (Pin_19)
- net E: now also J6.8 (Pin_8), U3.2 (A1); no longer J6.15 (Pin_15)
- net G1: now also J6.13 (Pin_13), U3.6 (A5); no longer J6.10 (Pin_10)
- net G2: now also J6.15 (Pin_15), U3.8 (A7); no longer J6.14 (Pin_14)
- net GND: now also C1.1, C2.1, J4.2 (Pin_2), J5.16, J5.4, R4.1, U1.B2A (SEL-), U1.H3 (H-), U1.S1 (SHIELD), U1.S2 (SHIELD), U1.S3 (SHIELD), U1.S4 (SHIELD), U1.V3 (V-), U2.10 (GND), U2.19 (/OE), U2.2 (A1), U2.3 (A2), U3.10 (GND), U3.19 (/OE)
- net JS_{s}: now also U1.B1A (SEL+)
- net JS_{x}: now also U1.H2 (H)
- net JS_{y}: now also U1.V2 (V)
- net LAT: now also J6.20 (Pin_20), U2.7 (A6); no longer J6.21 (Pin_21)
- net OE: now also J6.19 (Pin_19), U2.6 (A5); no longer J6.22 (Pin_22)
- net R1: now also J6.12 (Pin_12), U3.5 (A4); no longer J6.8 (Pin_8)
- net R2: now also J6.14 (Pin_14), U3.7 (A6); no longer J6.12 (Pin_12)
- net LED_G: now reaches J7.4 (Pin_4)
- net LED_G: now also R2.2
- net LED_B: now reaches J7.5 (Pin_5)
- net LED_B: now also R1.2
- net LED renamed LED_R
- net LED_R: now also R3.2
- new net: D1.4 (BK), R1.1
- new net: D2.C, R4.2
- new net: D1.3 (GK), R2.1
- new net: D1.2 (RK), R3.1
- new net M1_A: J5.9, U3.11 (B8)
- new net M1_B: J5.10, U2.11 (B8)
- new net M1_B1: J5.2, U3.16 (B3)
- new net M1_B2: J5.6, U3.17 (B2)
- new net M1_C: J5.11, U2.16 (B3)
- new net M1_CLK: J5.13, U2.15 (B4)
- new net M1_D: J5.12, U2.12 (B7)
- new net M1_E: J5.8, U3.18 (B1)
- new net M1_G1: J5.3, U3.14 (B5)
- new net M1_G2: J5.7, U3.12 (B7)
- new net M1_LAT: J5.14, U2.13 (B6)
- new net M1_OE: J5.15, U2.14 (B5)
- new net M1_R1: J5.1, U3.15 (B4)
- new net M1_R2: J5.5, U3.13 (B6)
- new net V5: C1.2, C2.2, D1.1 (A), J4.1 (Pin_1), J6.1 (Pin_1), J7.1 (Pin_1), SW1.1 (A), U2.1 (T/R), U2.20 (VCC), U3.1 (T/R), U3.20 (VCC)
- no-connect marks 38 -> 47
Other:
- note added: "Additional Peripherals"
- note added: "Joystick"
- note added: "LED Matrix"
- note added: "OLED Display"
- note added: "Power"
- note added: "RFID"
- moved on the sheet: J1, J2, J3, J6, J7

Commit message: pcb submission and update pins
Parts:
- U1: now left out of the parts list
Connections:
- net RFID_TX: now reaches J6.3 (Pin_3)
- net RFID_TX: now also J3.1 (Pin_1)
- net RFID_RX: now reaches J6.4 (Pin_4)
- net RFID_RX: now also J3.2 (Pin_2)
- net SCL: no longer names the net of J7.19 (Pin_19)
- net SCL: no longer J3.1 (Pin_1)
- net SDA: no longer names the net of J7.18 (Pin_18)
- net SDA: no longer J3.2 (Pin_2)
- net TX renamed OLED_TX
Changed lines of the file:
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@@
 	)
 	(junction
-		(at 45.72 129.54)
-		(diameter 0)
-		(color 0 0 0 0)
-	)
-	(junction
 		(at 57.15 129.54)
 		(diameter 0)
@@
 	)
 	(no_connect
-		(at 135.89 44.45)
-	)
-	(no_connect
 		(at 44.45 44.45)
 	)
@@
 	)
 	(no_connect
-		(at 130.81 44.45)
-	)
-	(no_connect
 		(at 54.61 219.71)
 	)
 	(no_connect
-		(at 97.79 71.12)
-	)
-	(no_connect
 		(at 123.19 71.12)
 	)
@@
 	)
 	(no_connect
+		(at 95.25 71.12)
+	)
+	(no_connect
 		(at 41.91 219.71)
 	)
@@
 	)
 	(no_connect
-		(at 133.35 44.45)
+		(at 135.89 44.45)
+	)
+	(no_connect
+		(at 97.79 71.12)
+	)
+	(no_connect
+		(at 92.71 71.12)
 	)
 	(no_connect
@@
 	(wire
 		(pts
-			(xy 64.77 226.06) (xy 64.77 219.71)
+			(xy 64.77 223.52) (xy 64.77 219.71)
 		)
 		(stroke
@@
 	(wire
 		(pts
-			(xy 45.72 129.54) (xy 44.45 129.54)
-		)
-		(stroke
-			(width 0)
-			(type default)
-		)
-	)
-	(wire
-		(pts
 			(xy 146.05 215.9) (xy 156.21 215.9)
 		)
@@
 	(wire
 		(pts
-			(xy 92.71 66.04) (xy 92.71 71.12)
-		)
-		(stroke
-			(width 0)
-			(type default)
-		)
-	)
-	(wire
-		(pts
 			(xy 142.24 213.36) (xy 156.21 213.36)
 		)
@@
 	(wire
 		(pts
+			(xy 130.81 36.83) (xy 130.81 44.45)
+		)
+		(stroke
+			(width 0)
+			(type default)
+		)
+	)
+	(wire
+		(pts
 			(xy 208.28 53.34) (xy 219.71 53.34)
 		)
@@
 	(wire
 		(pts
-			(xy 74.93 219.71) (xy 74.93 226.06)
+			(xy 74.93 219.71) (xy 74.93 223.52)
 		)
 		(stroke
@@
 	(wire
 		(pts
-			(xy 55.88 254) (xy 53.34 254)
+			(xy 133.35 39.37) (xy 133.35 44.45)
 		)
 		(stroke
@@
 	(wire
 		(pts
-			(xy 215.9 109.22) (xy 219.71 109.22)
+			(xy 55.88 254) (xy 53.34 254)
 		)
 		(stroke
@@
 	(wire
 		(pts
-			(xy 95.25 68.58) (xy 95.25 71.12)
+			(xy 215.9 109.22) (xy 219.71 109.22)
 		)
 		(stroke
@@
 		)
 	)
-	(label "SDA"
-		(at 95.25 68.58 0)
-		(effects
-			(font
-				(size 1.27 1.27)
-			)
-			(justify left bottom)
-		)
-	)
 	(label "R1"
 		(at 110.49 43.18 0)
@@
 		)
 	)
+	(label "RFID_RX"
+		(at 130.81 36.83 0)
+		(effects
+			(font
+				(size 1.27 1.27)
+			)
+			(justify left bottom)
+		)
+	)
 	(label "SCK"
 		(at 80.01 67.31 0)
@@
 		)
 	)
-	(label "TX"
+	(label "OLED_TX"
 		(at 82.55 69.85 0)
 		(effects
@@
 		)
 	)
-	(label "SCL"
+	(label "RFID_TX"
 		(at 109.22 217.17 0)
 		(effects
@@
 	)
 	(label "SCK"
-		(at 64.77 226.06 0)
+		(at 64.77 223.52 0)
 		(effects
 			(font
@@
 		)
 	)
-	(label "TX"
+	(label "OLED_TX"
 		(at 69.85 226.06 0)
 		(effects
@@
 	)
 	(label "CSn"
-		(at 74.93 226.06 0)
+		(at 74.93 223.52 0)
+		(effects
+			(font
+				(size 1.27 1.27)
+			)
+			(justify left bottom)
+		)
+	)
+	(label "RFID_TX"
+		(at 133.35 39.37 0)
 		(effects
 			(font
@@
 		)
 	)
-	(label "SCL"
-		(at 92.71 66.04 0)
-		(effects
-			(font
-				(size 1.27 1.27)
-			)
-			(justify left bottom)
-		)
-	)
 	(label "M1_C"
 		(at 278.13 68.58 180)
@@
 		)
 	)
-	(label "SDA"
+	(label "RFID_RX"
 		(at 106.68 214.63 0)
 		(effects
@@
 		(unit 1)
 		(exclude_from_sim no)
-		(in_bom yes)
+		(in_bom no)
 		(on_board yes)
 		(dnp no)
